File: hw/ctrl/v0.1/rwled-ctrl.kicad_sch (KiCad schematic)
At the start: 49 parts, among them J21 batt-chg, J31 USB_B_Micro, J61 led-a, J62 led-b, J63 led-c, J64 led-d, J65 batt-ab, J66 batt-cd, Q31 UMH3N, Q61 IRF4905STRLPBF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

Commit message: hw - архив доработанных и отправленных в заказ плат
Connections:
- net GND: now also Q63.1 (E1), Q64.1 (E1); no longer Q63.6 (C1), Q64.6 (C1)
- net at Q61.1 (G), R61.1: now also Q63.6 (C1); no longer Q63.1 (E1)
- net at R54.1: now also Q64.6 (C1); no longer Q64.1 (E1)
Changed lines of the file:
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@@
     )
   )
-  (symbol (lib_id "Transistor_BJT:UMH3N") (at 150.495 97.155 0) (mirror x) (unit 1)
-    (in_bom yes) (on_board yes) (dnp no)
-    (property "Reference" "Q63" (at 158.115 95.885 0)
+  (symbol (lib_id "Transistor_BJT:UMH3N") (at 150.495 97.155 0) (unit 1)
+    (in_bom yes) (on_board yes) (dnp no)
+    (property "Reference" "Q63" (at 158.115 96.52 0)
       (effects (font (size 1.27 1.27)) (justify left))
     )
@@
       (effects (font (size 1.27 1.27)) (justify left))
     )
-    (property "Footprint" "Package_TO_SOT_SMD:SOT-363_SC-70-6" (at 150.622 85.979 0)
+    (property "Footprint" "Package_TO_SOT_SMD:SOT-363_SC-70-6" (at 150.622 108.331 0)
       (effects (font (size 1.27 1.27)) hide)
     )
@@
     )
   )
-  (symbol (lib_id "Transistor_BJT:UMH3N") (at 33.02 151.13 0) (mirror x) (unit 1)
-    (in_bom yes) (on_board yes) (dnp no)
-    (property "Reference" "Q64" (at 40.64 149.86 0)
+  (symbol (lib_id "Transistor_BJT:UMH3N") (at 33.02 151.13 0) (unit 1)
+    (in_bom yes) (on_board yes) (dnp no)
+    (property "Reference" "Q64" (at 40.64 150.495 0)
       (effects (font (size 1.27 1.27)) (justify left))
     )
@@
       (effects (font (size 1.27 1.27)) (justify left))
     )
-    (property "Footprint" "Package_TO_SOT_SMD:SOT-363_SC-70-6" (at 33.147 139.954 0)
-      (effects (font (size 1.27 1.27)) hide)
-    )
+    (property "Footprint" "Package_TO_SOT_SMD:SOT-363_SC-70-6" (at 33.147 162.306 0)
+      (effects (font (size 1.27 1.27)) hide)
+    )
